Commit message: 更新

File: src/panda_moveit_config/config/panda_arm_hand.srdf.xacro (robot description, xacro)
@@ -23,6 +23,6 @@
   </group_state>
   <group_state name="close" group="hand">
-    <joint name="panda_finger_joint1" value="0" />
-    <joint name="panda_finger_joint2" value="0" />
+    <joint name="panda_finger_joint1" value="0.0" />
+    <joint name="panda_finger_joint2" value="0.0" />
   </group_state>
   <!--END EFFECTOR: Purpose: Represent information about an end effector.-->

File: src/robot_description/urdf/panda.urdf (robot description, URDF)
Before this commit: robot panda, 14 links, 13 joints
Joints:
- joint panda_finger_joint1: limit lower=0.0 upper=0.04 effort=40 velocity=0.2 -> lower=0.0 upper=0.04 effort=40.0 velocity=100.0
- joint panda_finger_joint2: limit lower=0.0 upper=0.04 effort=40 velocity=0.2 -> lower=0.0 upper=0.04 effort=40.0 velocity=100.0
