Commit message: 移植好GraphExecuter，并修复夹爪无法抓取的bug

File: ros2_project/src/panda_moveit_config/config/panda.urdf.xacro (robot description, xacro)
@@ -1,39 +1,42 @@
 <?xml version="1.0"?>
 <robot xmlns:xacro="http://www.ros.org/wiki/xacro" name="panda">
-    <xacro:arg name="initial_positions_file" default="initial_positions.yaml" />
-    <xacro:arg name="ros2_control_hardware_type" default="mock_components" />
+    <xacro:arg name="initial_positions_file" default="$(find panda_moveit_config)/config/initial_positions.yaml"/>
     <xacro:property name="PI" value="3.14159274"/>
     <!-- Import panda urdf file -->
-    <xacro:include filename="$(find robot_description)/urdf/panda.urdf" />
+    <xacro:include filename="$(find robot_description)/urdf/panda.urdf"/>
+    <!-- Lidar -->
+    <!-- <xacro:include filename="$(find robot_description)/urdf/lidar/lidar.xacro"/>
+    <xacro:lidar_v0 parent="panda_link7">
+        <origin xyz="-0.2 -0.2 0.2" rpy="0 ${PI/2} 0"/>
+    </xacro:lidar_v0> -->
     <xacro:include filename="$(find robot_description)/urdf/camera/camera.xacro"/>
     <!-- Camera -->
     <xacro:camera_v0 parent="panda_link0">
-	    <origin xyz="0.2 0.6 0.7" rpy="0 ${PI/2} 0"/>
+        <origin xyz="0.2 0.6 0.7" rpy="0 ${PI/2} 0"/>
     </xacro:camera_v0>
     <xacro:camera_gazebo_v0/>
-    <!-- controllers for gazebo -->
-    <xacro:include filename="panda.gazebo_ros2_control.xacro" />
-    <xacro:panda_gazebo_ros2_control initial_positions_file="$(arg initial_positions_file)"/>
-    <!-- There were no gazebo files in the original file-->
-  <gazebo>
-    <plugin
+    <gazebo>
+        <plugin
         filename="gz_ros2_control-system"
         name="gz_ros2_control::GazeboSimROS2ControlPlugin">
-        <parameters>$(find panda_moveit_config)/config/ros2_controllers.yaml</parameters>
-    </plugin>
-    <plugin
+            <parameters>$(find panda_moveit_config)/config/ros2_controllers.yaml</parameters>
+        </plugin>
+        <plugin
         filename="gz-sim-joint-state-publisher-system"
         name="gz::sim::systems::JointStatePublisher">
     </plugin>
-    <plugin
+        <plugin
         filename="gz-sim-pose-publisher-system"
         name="gz::sim::systems::PosePublisher">
-        <publish_link_pose>true</publish_link_pose>
-        <use_pose_vector_msg>true</use_pose_vector_msg>
-        <publish_nested_model_pose>true</publish_nested_model_pose>
-    </plugin>
-    <plugin filename="ignition-gazebo-sensors-system" name="ignition::gazebo::systems::Sensors">
-      <render_engine>ogre2</render_engine>
-    </plugin>
-  </gazebo>
+            <publish_link_pose>true</publish_link_pose>
+            <use_pose_vector_msg>true</use_pose_vector_msg>
+            <publish_nested_model_pose>true</publish_nested_model_pose>
+        </plugin>
+        <plugin filename="ignition-gazebo-sensors-system" name="ignition::gazebo::systems::Sensors">
+            <render_engine>ogre2</render_engine>
+        </plugin>
+    </gazebo>
+    <xacro:include filename="panda.gazebo.ros2_control.xacro" />
+    <xacro:panda_gazebo_ros2_control name="GazeboSimSystem"
+        initial_positions_file="$(arg initial_positions_file)"/>
 </robot>

File: ros2_project/src/robot_description/urdf/camera/camera.xacro (robot description, xacro)
@@ -1,28 +1,28 @@
 <?xml version="1.0"?>
 <robot name="delirobo" xmlns:xacro="http://ros.org/wiki/xacro">
-  <xacro:include filename="$(find robot_description)/urdf/camera/camera.gazebo"/>
-  <xacro:macro name="camera_v0" params="parent *joint_origin">
-	<joint name="camera_joint" type="fixed">
-	  <xacro:insert_block name="joint_origin"/>
-	  <parent link="${parent}"/>
-	  <child link="camera_link"/>
-	</joint>
-	<link name="camera_link">
-	  <visual>
-		<geometry>
-		  <mesh filename="package://robot_description/meshes/visual/camera.dae"/>
-		</geometry>
-	  </visual>
-	  <collision>
-		<geometry>
-		  <mesh filename="package://robot_description/meshes/collision/camera.stl"/>
-		</geometry>
-	  </collision>
-	  <inertial>
-		<origin xyz="0 0 0"/>
-		<mass value="0.1"/>
-		<inertia ixx="0.00001" ixy="0" ixz="0" iyy="0.00001" iyz="0" izz="0.00001" />
-	  </inertial>
-	</link>
-  </xacro:macro>
+	<xacro:include filename="$(find robot_description)/urdf/camera/camera.gazebo"/>
+	<xacro:macro name="camera_v0" params="parent *joint_origin">
+		<joint name="camera_joint" type="fixed">
+			<xacro:insert_block name="joint_origin"/>
+			<parent link="${parent}"/>
+			<child link="camera_link"/>
+		</joint>
+		<link name="camera_link">
+			<visual>
+				<geometry>
+					<mesh filename="package://robot_description/meshes/visual/camera.dae"/>
+				</geometry>
+			</visual>
+			<collision>
+				<geometry>
+					<mesh filename="package://robot_description/meshes/collision/camera.stl"/>
+				</geometry>
+			</collision>
+			<inertial>
+				<origin xyz="0 0 0"/>
+				<mass value="0.1"/>
+				<inertia ixx="0.00001" ixy="0" ixz="0" iyy="0.00001" iyz="0" izz="0.00001" />
+			</inertial>
+		</link>
+	</xacro:macro>
 </robot>

File: ros2_project/src/robot_description/urdf/panda.urdf (robot description, URDF)
Before this commit: robot panda, 14 links, 13 joints
Links:
- removed link random
Joints:
- removed joint panda_finger_joint2_mimic
